File: green_house.kicad_pcb (KiCad board)
At the start: 2 copper layers, 38 parts, among them J1 Conn_01x02_Female, J2 WATER-PUMP, J3 Conn_01x02_Female, J4 MOTOR-1, J5 MOTOR-2, K1 SANYOU_SRD_Form_C, K2 SANYOU_SRD_Form_C, Q1 TIP122, Q2 TIP122, Q3 TIP122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

Commit message: fixed pads and holes dimensions
Parts:
- removed J1: Conn_01x02_Female, TestPoint:TestPoint_2Pads_Pitch5.08mm_Drill1.3mm
- added ?: , , F.Cu at (40.6, 68.6)
- added ?: , , F.Cu at (35.6, 68.6)
Routing:
- net GND: track 844.4 -> 842.5 mm
